File: hardware/schematics/schematics.kicad_sch (KiCad schematic)
At the start: 20 parts, among them J1 Conn_01x02, M1 Micro Servo Motor, SW1 One_SW, SW2 Two_SW, SW3 Enter_SW, SW4 Reset_SW

Commit message: Fix schematics.pdf
Other:
- company: Tomoya Yoshii -> Tomoya Y
Changed lines of the file:
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@@
 		(title "Arduino Dual-Lock Safe")
 		(date "2025/12/04")
-		(company "Tomoya Yoshii")
+		(company "Tomoya Y")
 	)
 	(junction
